File: toshiba-64mbit-adapter.sch (KiCad schematic (older format))
At the start: 9 parts, among them U1 TC5364205, U2 W29GL064C, U3 74HCT244, U4 74HCT244, U5 74HCT244, U6 74HCT244, U7 74HCT244, U8 TPS73633DBV

Commit message: Updated to current KiCad stable
- Updated project files to current KiCad stable version
- Added gitignore to ignore backup files
Parts:
- U3, U4, U5, U6, U7: symbol 74xx:74HCT244 -> toshiba-64mbit-adapter-rescue:74HCT244-74xx
Changed lines of the file:
@@
 EESchema Schematic File Version 4
-LIBS:toshiba-64mbit-adapter-cache
-EELAYER 29 0
+EELAYER 30 0
 EELAYER END
 $Descr A4 11693 8268
@@
 	2650 2600 2900 2600
 $Comp
-L 74xx:74HCT244 U4
+L toshiba-64mbit-adapter-rescue:74HCT244-74xx U4
 U 1 1 5C861A2E
 P 6350 3350
@@
 $EndComp
 $Comp
-L 74xx:74HCT244 U5
+L toshiba-64mbit-adapter-rescue:74HCT244-74xx U5
 U 1 1 5C8634EA
 P 7950 3350
@@
 $EndComp
 $Comp
-L 74xx:74HCT244 U7
+L toshiba-64mbit-adapter-rescue:74HCT244-74xx U7
 U 1 1 5C863DE8
 P 9400 3350
@@
 $EndComp
 $Comp
-L 74xx:74HCT244 U3
+L toshiba-64mbit-adapter-rescue:74HCT244-74xx U3
 U 1 1 5C865388
 P 6300 5450
@@
 $EndComp
 $Comp
-L 74xx:74HCT244 U6
+L toshiba-64mbit-adapter-rescue:74HCT244-74xx U6
 U 1 1 5C865EC6
 P 8000 5400

Commit message: Labeling
- A11 label on DIP42 is now bold to match other labels
- Renamed U2 to indicate newer, more common parts
Parts:
- U2: value W29GL064C -> S29*L
Changed lines of the file:
@@
 	1    0    0    -1
 $EndComp
-Text Label 2900 2500 2    50   ~ 0
+Text Label 2900 2500 2    50   ~ 10
 A21
 $Comp
@@
 P 1450 5350
 F 0 "U2" H 1700 6575 50  0000 C CNN
-F 1 "W29GL064C" H 1700 6484 50  0000 C CNN
+F 1 "S29*L" H 1700 6484 50  0000 C CNN
 F 2 "Package_SO:TSOP-I-48_18.4x12mm_P0.5mm" H 1450 5350 50  0001 C CNN
 F 3 "" H 1450 5350 50  0001 C CNN

Commit message: Project setup
- Updated schematic page settings with title, ref, license
- Added some notes to parts and a link to a doc with a pinout for the 64Mbit Toshiba chip
- Updated plots
Parts:
- U2: Notes (none) -> Use with S29GL064N, S29GL032N, S29AL016J, S29AL008J, or fun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
Changed lines of the file:
@@
 encoding utf-8
 Sheet 1 1
-Title ""
-Date ""
-Rev ""
+Title "Flash to Toshiba Mask ROM Adapter"
+Date "2020-10-16"
+Rev "1.2"
 Comp ""
-Comment1 ""
-Comment2 ""
+Comment1 "License: CC0 1.0 Universal"
+Comment2 "https://github.com/tdaede/toshiba-64mbit-adapter"
 Comment3 ""
 Comment4 ""
@@
 F 1 "TC5364205" H 3250 3734 50  0000 C CNN
 F 2 "Package_DIP:DIP-42_W15.24mm" H 3000 2550 50  0001 C CNN
-F 3 "" H 3000 2550 50  0001 C CNN
+F 3 "https://smitdogg.mameworld.info/du/romref.txt" H 3000 2550 50  0001 C CNN
 	1    3000 2550
 	1    0    0    -1
@@
 F 2 "Package_SO:TSOP-I-48_18.4x12mm_P0.5mm" H 1450 5350 50  0001 C CNN
 F 3 "" H 1450 5350 50  0001 C CNN
+F 4 "Use with S29GL064N, S29GL032N, S29AL016J, S29AL008J, or functionally identical NOR flash " H 1450 5350 50  0001 C CNN "Notes"
 	1    1450 5350
 	1    0    0    -1
