File: 8bit/toshiba-64mbit-adapter.kicad_pcb (KiCad board)
At the start: 2 copper layers, 18 x 55 mm, 9 parts, among them U1 TC5364205, U2 W29GL064C, U3 74HCT244, U4 74HCT244, U5 74HCT244, U6 74HCT244, U7 74HCT244, U8 TPS73633DBV

Commit message: split to separate version
going to do this as 8bit and 16bit versions rather than a single configurable version
Other:
- board text added: "CC0 v1.1 2019"
- board text removed: "CC0 v1.0 2019"
Changed lines of the file:
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@@
   )
   (gr_circle (center 124.4 76.6) (end 124.6 76.6) (layer F.SilkS) (width 0.12))
-  (gr_text "CC0 v1.0 2019" (at 113.3 87.05 270) (layer B.SilkS)
+  (gr_text "CC0 v1.1 2019" (at 113.3 87.05 270) (layer B.SilkS)
     (effects (font (size 1 1) (thickness 0.15)) (justify mirror))
   )

Commit message: this probably works
Parts:
- U2: value W29GL064C -> S29*L
- U3, U4, U5: value 74HCT244 -> 74LVC244APW,118
Connections:
- U1 pad 30: /D15 -> /A-1
- U2 pad 45: /md15 -> /ma-1
- U2 pad 47: +3V3 -> GND
- U5 pad 17: GND -> /A-1
- U5 pad 3: Net-(U5-Pad3) -> /ma-1
- U6 pad 12: /D15 -> GND
- U6 pad 20: +3V3 -> +5V
- U6 pad 8: /md15 -> GND
- U7 pad 20: +3V3 -> +5V
Routing:
- net +5V: track 7.75 -> 25.0 mm, vias 0 -> 2
- net /ma-1: track 0.00 -> 15.4 mm, vias 0 -> 1
- net /md15: track 10.7 -> 0.00 mm, vias 1 -> 0
- net /A-1: track 0.00 -> 8.99 mm, vias 0 -> 1
- net /D15: track 5.31 -> 0.00 mm
- net +3V3: track 11.9 -> 8.38 mm, vias 5 -> 4
- net GND: track 9.87 -> 10.9 mm
