File: 8bit/toshiba-64mbit-adapter.sch (KiCad schematic (older format))
At the start: 9 parts, among them U1 TC5364205, U2 S29*L, U3 74LVC244APW,118, U4 74LVC244APW,118, U5 74LVC244APW,118, U6 74HCT244, U7 74HCT244, U8 TPS73633DBV

Commit message: this probably works
Connections:
- net +3V3: no longer U2.47 (/BYTE)
- net GND: now also U2.47 (/BYTE), U6.12 (1Y3), U6.8 (1A3); no longer U5.17 (2A0)
- net ma-1: now reaches U5.3 (2Y0)
- net ma-1: now also U2.45 (DQ15)
- net D15 renamed A-1
- net A-1: now also U5.17 (2A0); no longer U6.12 (1Y3)
- removed net md15: U2.45 (DQ15), U6.8 (1A3)
Changed lines of the file:
@@
 A20
 Text Label 3600 2700 0    50   ~ 10
-D15
+A-1
 Text Label 3600 2900 0    50   ~ 10
 D14
@@
 ma15
 Text Label 2050 4650 0    50   ~ 0
-md15
+ma-1
 Text Label 2050 4750 0    50   ~ 0
 md7
@@
 Wire Wire Line
 	2050 4550 2450 4550
-$Comp
-L power:+3V3 #PWR0115
-U 1 1 5C8A68FE
-P 2450 4450
-F 0 "#PWR0115" H 2450 4300 50  0001 C CNN
-F 1 "+3V3" H 2465 4623 50  0000 C CNN
-F 2 "" H 2450 4450 50  0001 C CNN
-F 3 "" H 2450 4450 50  0001 C CNN
-	1    2450 4450
-	1    0    0    -1
-$EndComp
 Wire Wire Line
 	2050 4450 2450 4450
@@
 Text Label 6800 4550 0    50   ~ 0
 D9
-Text Label 6800 4450 0    50   ~ 0
-D15
 Text Label 6800 4350 0    50   ~ 0
 D7
@@
 Connection ~ 9700 2750
 Connection ~ 9200 2450
-Wire Wire Line
-	9050 2450 9200 2450
 Text Label 9200 1550 2    50   ~ 0
 E
@@
 Text Label 5800 4350 2    50   ~ 0
 md7
-Text Label 5800 4450 2    50   ~ 0
-md15
 Text Label 5800 4550 2    50   ~ 0
 md9
@@
 	1    0    0    -1
 $EndComp
-Wire Wire Line
-	9200 1850 9050 1850
-Wire Wire Line
-	9050 1850 9050 2450
 $Comp
 L power:+3V3 #PWR0121
@@
 	1    0    0    -1
 $EndComp
+Wire Wire Line
+	2450 4450 2450 4550
+Connection ~ 2450 4550
+Text Label 9200 1850 2    50   ~ 0
+A-1
+Text Label 10200 1850 0    50   ~ 0
+ma-1
+Wire Wire Line
+	5800 4450 5600 4450
+Wire Wire Line
+	5600 4450 5600 5450
+Wire Wire Line
+	5600 5450 6300 5450
+Connection ~ 6300 5450
+Wire Wire Line
+	6800 4450 6950 4450
+Wire Wire Line
+	6950 4450 6950 5450
+Wire Wire Line
+	6950 5450 6300 5450
 $EndSCHEMATC
